File: PCB/splitkeyboard.kicad_pcb (KiCad board)
At the start: 2 copper layers, 287 x 126.2 mm, 118 parts, among them SW1 SW_Push, SW10 SW_Push, SW11 SW_Push, SW12 SW_Push, SW13 SW_Push, SW14 SW_Push, SW15 SW_Push, SW16 SW_Push, SW17 SW_Push, SW18 SW_Push, SW19 SW_Push, SW2 SW_Push, SW20 SW_Push, SW21 SW_Push, SW22 SW_Push, SW23 SW_Push, SW24 SW_Push, SW25 SW_Push, SW26 SW_Push, SW27 SW_Push, SW28 SW_Push, SW29 SW_Push, SW3 SW_Push, SW30 SW_Push, SW31 SW_Push, SW32 SW_Push, SW33 SW_Push, SW34 SW_Push, SW35 SW_Push, SW36 SW_Push, SW37 SW_Push, SW38 SW_Push, SW39 SW_Push, SW4 SW_Push, SW40 SW_Push, SW41 SW_Push, SW42 SW_Push, SW43 SW_Push, SW44 SW_Push, SW45 SW_Push, SW46 SW_Push, SW47 SW_Push, SW48 SW_Push, SW49 SW_Push, SW5 SW_Push, SW50 SW_Push, SW51 SW_Push, SW52 SW_Push, SW6 SW_Push, SW7 SW_Push, SW8 SW_Push, SW9 SW_Push, U1 XIAO-nRF52840-SMD, U2 XIAO-nRF52840-SMD

Commit message: Add files via upload
Parts:
- TP1, TP2, TP3, TP4: moved to B.Cu
- moved R2 1.92 mm to (312.3, 133.7), turned to -90 degrees
- moved R1 1.81 mm to (314.9, 133.8), turned to 90 degrees
- turned TP1 to 180 degrees
- turned TP2 to 180 degrees
- turned TP3 to 180 degrees
- turned TP4 to 180 degrees
Routing:
- net /right/COL4: track 203.9 -> 207.7 mm
- net /left/BT_PIN: track 36.0 -> 33.2 mm
- net /right/VBAT: track 58.4 -> 59.4 mm, vias 1 -> 2
- net GND: track 120.7 -> 121.3 mm
